File: keyboard.kicad_sch (KiCad schematic)
At the start: 100 parts

Commit message: wireless
Parts:
- removed C10, C11, C12, C13, C14, C15, C16, C17, C18, C3, C4, C5, C6, C7, C8, C9: (no value), symbol Device:C
- removed D1, D10, D11, D12, D13, D14, D15, D16, D17, D19, D2, D20, D21, D22, D23, D3, D4, D5, D6, D7, D8, D9: (no value), symbol Device:D_Small
- removed D33, D34, D35, D36, D37, D38, D39, D40: (no value), symbol LED:WS2812B
- removed J2: (no value), symbol Connector:AudioJack4
- removed SW25: (no value), symbol kbd:SW_PUSH
- added J2: Conn_01x02, hb44:TH_BatteryConn, symbol Connector_Generic:Conn_01x02
- added J3: Conn_01x05, hb44:Pimoroni Haptic Buzz DRV2605L Driver, symbol Connector_Generic:Conn_01x05
- added JP5, JP6: SolderJumper_3_Open, keyswitches:jumperClean, symbol Jumper:SolderJumper_3_Open
- added SW25: SW_DPDT_x2, Button_Switch_SMD:SW_SPDT_PCM12, symbol Switch:SW_DPDT_x2
- C1, C19, C2, C20: value (none) -> 10n; footprint (none) -> keyswitches:Cap_0603_Clean
- D1: renamed from D18; value (none) -> (none); footprint (none) -> hb44:SMD_SOD123
- D2: renamed from D24; value (none) -> WS2812B+Cap; footprint (none) -> hb44:SMD_WS2812B+Cap0603; symbol LED:WS2812B -> hb44:WS2812B+Cap
- D3: renamed from D25; value (none) -> WS2812B+Cap; footprint (none) -> hb44:SMD_WS2812B+Cap0603; symbol LED:WS2812B -> hb44:WS2812B+Cap
- D4: renamed from D26; value (none) -> WS2812B+Cap; footprint (none) -> hb44:SMD_WS2812B+Cap0603; symbol LED:WS2812B -> hb44:WS2812B+Cap
- D5: renamed from D27; value (none) -> WS2812B+Cap; footprint (none) -> hb44:SMD_WS2812B+Cap0603; symbol LED:WS2812B -> hb44:WS2812B+Cap
- D6: renamed from D28; value (none) -> WS2812B+Cap; footprint (none) -> hb44:SMD_WS2812B+Cap0603; symbol LED:WS2812B -> hb44:WS2812B+Cap
- D7: renamed from D29; value (none) -> WS2812B+Cap; footprint (none) -> hb44:SMD_WS2812B+Cap0603; symbol LED:WS2812B -> hb44:WS2812B+Cap
- D8: renamed from D30; value (none) -> WS2812B+Cap; footprint (none) -> hb44:SMD_WS2812B+Cap0603; symbol LED:WS2812B -> hb44:WS2812B+Cap
- D9: renamed from D31; value (none) -> WS2812B+Cap; footprint (none) -> hb44:SMD_WS2812B+Cap0603; symbol LED:WS2812B -> hb44:WS2812B+Cap
- J1: value (none) -> AudioJack4; footprint (none) -> hb44:SMD_3.5mm_TRRS
- JP1, JP2, JP3, JP4: value (none) -> SolderJumper_3_Open; footprint (none) -> keyswitches:jumperClean
- LCD1: renamed from OL1; value (none) -> nice!view; footprint (none) -> hb44:nice!view; symbol kbd:OLED -> hb44:nice!view
- R1, R2, R3, R4, R5, R6, R7, R8: value (none) -> 10k; footprint (none) -> keyswitches:Res_1206_Clean
- SW1, SW10, SW11, SW12, SW13, SW14, SW15, SW16, SW17, SW19, SW2, SW20, SW21, SW22, SW23, SW3, SW4, SW5, SW6, SW7, SW8, SW9: value (none) -> Switch+Diode; footprint (none) -> hb44:SMD_CherryMX_MidHeight_Choc_HotSwap+SOD123; symbol MX_Alps_Hybrid:MX-NoLED -> hb44:Switch+Diode
- SW18: value (none) -> RotaryEncoder_Switch; footprint (none) -> keyswitches:ec11
- SW24: value (none) -> SW_PUSH; footprint (none) -> hb44:SMD_SW_PUSH
- U1: value (none) -> nice!nano; footprint (none) -> hb44:nice!nano; symbol kbd:ProMicro -> hb44:nice!nano
Connections:
- net GND: now also JP2.3 (B), JP3.1 (A), J2.1 (Pin_1), JP5.3 (B), JP6.1 (A); no longer JP1.3 (B), JP4.1 (A)
- net SCL: now also U1.8 (P0.24/H), J3.3 (Pin_3); no longer JP2.1 (A), JP3.3 (B), U1.6 (3/D0/SCL)
- net SDA: now also U1.7 (P0.22/H), J3.2 (Pin_2), J3.4 (Pin_4); no longer JP1.1 (A), JP4.3 (B), U1.5 (2/D1/SDA)
- net VCC: now also LCD1.3 (VCC), JP5.1 (A), JP6.3 (B); no longer JP2.3 (B), JP3.1 (A)
- net rotA: now also U1.20 (P0.31/L); no longer U1.7 (4/D4)
- net rotB: now also U1.19 (P0.29/L); no longer U1.8 (5/C6)
- net row0: now also SW1.3, SW2.3, SW3.3, SW4.3, SW5.3, SW6.3
- net row1: now also SW10.3, SW11.3, SW12.3, SW7.3, SW8.3, SW9.3
- net row2: now also SW13.3, SW14.3, SW15.3, SW16.3, SW17.3
- net row3: now also SW19.3, SW20.3, SW21.3, SW22.3, SW23.3
- net RAW: now reaches U1.24 (BAT+)
- net RAW: now also SW25.2 (B)
- net Data renamed CS
- net CS: now also JP1.3 (B), JP4.1 (A)
- net OLED_1 renamed LCD_1
- net OLED_2 renamed LCD_2
- net OLED_3 renamed LCD_4
- net LCD_4: now also LCD1.4 (GND); no longer LCD1.3 (VCC)
- net OLED_4 renamed LCD_5
- net LCD_5: now also LCD1.5 (CS); no longer LCD1.4 (GND)
- new net: J2.2 (Pin_2), SW25.3 (C)
- new net HAP_1: J3.1 (Pin_1), JP5.2 (C)
- new net HAP_5: J3.5 (Pin_5), JP6.2 (C)
- new net MOSI: JP1.1 (A), JP4.3 (B), U1.5 (P0.17/H)
- new net SCK: JP2.1 (A), JP3.3 (B), U1.6 (P0.20/H)
- no-connect marks 7 -> 3
Other:
- note added: "-160x68 resolution using SPI protocol -Displays status and customizable graphics"
- note added: "-4x6 matrix, 23 switches -Hotswap MX/Choc footprint"
- note added: "-Allows battery to be turned off -Useful for travel"
- note added: "-DRV2605L I2C haptic driver -ELV1411A linear resonant actuator"
- note added: "-Resets the microcontroller -Located at the top"
- note added: "Battery Switch"
- note added: "Haptic Feedback"
- note added: "LCD Status Display"
- note removed: "-128x32 resolution using I2C protocol -Displays status and customizable graphics"
- note removed: "-4x6 matrix, 23 switches -Utilizes a hotswap optional footprint"
- note removed: "-Resets the microcontroller -Located on the back"
- note removed: "OLED Status Display"
