File: PCB/keyboard.kicad_pcb (KiCad board)
At the start: 2 copper layers, 131.8 x 123.7 mm, 69 parts, among them J2 Conn_01x02, J3 Conn_01x05, Q1 Q_PMOS_GSD, SW1 Switch+Diode, SW10 Switch+Diode, SW11 Switch+Diode, SW12 Switch+Diode, SW13 Switch+Diode, SW14 Switch+Diode, SW15 Switch+Diode, SW16 RotaryEncoder_Switch, SW17 Switch+Diode, SW18 Switch+Diode, SW19 Switch+Diode, SW2 Switch+Diode, SW20 Switch+Diode, SW21 Switch+Diode, SW24 SW_PUSH, SW25 SW_DPDT_x2, SW3 Switch+Diode, SW4 Switch+Diode, SW5 Switch+Diode, SW6 Switch+Diode, SW7 Switch+Diode, SW8 Switch+Diode, SW9 Switch+Diode, U1 ProMicro_r, U2 74AUP2G14

Commit message: vertical
Parts:
- removed JP1, JP2, JP3, JP4, JP5, JP6: SolderJumper_3_Open, hb44:jumperClean
- removed SW24: SW_PUSH, hb44:SMD_SW_SPST_B3U-3000P-B
- removed SW25: SW_DPDT_x2, hb44:SMD_SW_SPDT_PCM12
- added C1: 0.1u, hb44:SMD_Cap_0603, B.Cu at (134.4, 40.9)
- added C10: 0.1u, hb44:SMD_Cap_0603, B.Cu at (46.2, 72.0)
- added C11: 0.1u, hb44:SMD_Cap_0603, B.Cu at (46.2, 91.0)
- added C12: 0.1u, hb44:SMD_Cap_0603, B.Cu at (48.7, 99.0)
- added C13: 0.1u, hb44:SMD_Cap_0603, B.Cu at (67.3, 101.9)
- added C14: 0.1u, hb44:SMD_Cap_0603, B.Cu at (86.7, 103.7)
- added C15: 0.1u, hb44:SMD_Cap_0603, B.Cu at (101.6, 111.1)
- added C16: 0.1u, hb44:SMD_Cap_0603, B.Cu at (114.8, 113.2)
- added C17: 0.1u, hb44:SMD_Cap_0603, B.Cu at (131.9, 117.9)
- added C18: 0.1u, hb44:SMD_Cap_0603, B.Cu at (147.2, 129.5)
- added C19: 0.1u, hb44:SMD_Cap_0603, B.Cu at (156.3, 146.7)
- added C2: 0.1u, hb44:SMD_Cap_0603, B.Cu at (124.3, 40.1)
- added C20: 0.1u, hb44:SMD_Cap_0603, B.Cu at (169.6, 146.9)
- added C21: 0.1u, hb44:SMD_Cap_0603, B.Cu at (168.4, 138.7)
- added C22: 0.1u, hb44:SMD_Cap_0603, B.Cu at (155.3, 117.8)
- added C23: 0.1u, hb44:SMD_Cap_0603, B.Cu at (158.1, 119.1)
- added C24: 0.1u, hb44:SMD_Cap_0603, B.Cu at (159.3, 120.4)
- added C25: 0.1u, hb44:SMD_Cap_0603, B.Cu at (154.9, 56.8)
- added C3: 0.1u, hb44:SMD_Cap_0603, B.Cu at (115.6, 33.9)
- added C4: 0.1u, hb44:SMD_Cap_0603, B.Cu at (110.8, 32.5)
- added C5: 0.1u, hb44:SMD_Cap_0603, B.Cu at (85.6, 30.8)
- added C6: 0.1u, hb44:SMD_Cap_0603, B.Cu at (75.4, 33.1)
- added C7: 0.1u, hb44:SMD_Cap_0603, B.Cu at (63.4, 38.5)
- added C8: 0.1u, hb44:SMD_Cap_0603, B.Cu at (47.9, 44.9)
- added C9: 0.1u, hb44:SMD_Cap_0603, B.Cu at (46.2, 54.0)
- added D1: , hb44:SMD_SOD123, B.Cu at (77.2, 60.7)
- added D10: , hb44:SMD_SOD123, B.Cu at (81.4, 47.7)
- added D11: , hb44:SMD_SOD123, B.Cu at (77.2, 47.7)
- added D12: , hb44:SMD_SOD123, B.Cu at (77.2, 80.2)
- added D13: , hb44:SMD_SOD123, B.Cu at (85.6, 80.2)
- added D14: , hb44:SMD_SOD123, B.Cu at (85.6, 47.7)
- added D15: , hb44:SMD_SOD123, B.Cu at (81.4, 60.7)
- added D17: , hb44:SMD_SOD123, B.Cu at (81.4, 41.2)
- added D18: , hb44:SMD_SOD123, B.Cu at (81.4, 54.2)
- added D19: , hb44:SMD_SOD123, B.Cu at (81.4, 67.2)
- added D2: , hb44:SMD_SOD123, B.Cu at (77.2, 67.2)
- added D20: , hb44:SMD_SOD123, B.Cu at (81.4, 80.2)
- added D21: , hb44:SMD_SOD123, B.Cu at (81.4, 73.7)
- added D3: , hb44:SMD_SOD123, B.Cu at (85.6, 67.2)
- added D4: , hb44:SMD_SOD123, B.Cu at (85.6, 60.7)
- added D5: , hb44:SMD_SOD123, B.Cu at (85.6, 41.2)
- added D6: , hb44:SMD_SOD123, B.Cu at (77.2, 54.2)
- added D7: , hb44:SMD_SOD123, B.Cu at (77.2, 73.7)
- added D8: , hb44:SMD_SOD123, B.Cu at (85.6, 73.7)
- added D9: , hb44:SMD_SOD123, B.Cu at (85.6, 54.2)
- added H4: MountingHole, hb44:MountingHole_4mm, F.Cu at (47.5, 81.5)
- added H5: MountingHole, hb44:MountingHole_4mm, F.Cu at (119.8, 110.7)
- added H6: MountingHole, hb44:MountingHole_4mm, F.Cu at (139.3, 117.6)
- added H7: MountingHole, hb44:MountingHole_4mm, F.Cu at (153.5, 133.1)
- added H8: MountingHole, hb44:MountingHole_4mm, F.Cu at (128.3, 57.7)
- added LED23: SK6812, hb44:SK6812-SIDE, B.Cu at (155.4, 90.5)
- added LED24: SK6812, hb44:SK6812-SIDE, B.Cu at (155.4, 69.5)
- added LED25: SK6812, hb44:SK6812-SIDE, B.Cu at (155.4, 53.3)
- added SW43: SW_DPDT_x2, hb44:SMD_SW_SPDT_PCM12, B.Cu at (103.8, 31.6)
- added SW44: SW_PUSH, hb44:SMD_SW_SPST_B3U-3000P-B, B.Cu at (116.1, 30.4)
- C26: renamed from C1; footprint hb44:Cap_0603_Clean -> hb44:SMD_Cap_0603
- C27: renamed from C2; footprint hb44:Cap_0603_Clean -> hb44:SMD_Cap_0603
- J1: renamed from J3; footprint hb44:Pimoroni Haptic Buzz DRV2605L Driver -> hb44:Pimoroni Haptic Buzz
- J2, R5, R6: moved to B.Cu
- LED1, LED10, LED11, LED12, LED13, LED14, LED15, LED16, LED17, LED18, LED19, LED2, LED20, LED21, LED22, LED3, LED4, LED5, LED6, LED7, LED8, LED9: value 0.1u -> SK6812; footprint hb44:SK6812-SIDE + 1608m Cap -> hb44:SK6812-SIDE; moved to B.Cu
- Q1: footprint hb44:SMD_P_MOSTFET_SOT-23 -> hb44:SMD_P_MOSFET_SOT-23; moved to B.Cu
- R1, R2, R3, R4: footprint hb44:Res_1206_Clean -> hb44:SMD_Res_1206
- SW1, SW10, SW11, SW12, SW13, SW14, SW17, SW18, SW19, SW2, SW20, SW21, SW3, SW4, SW6, SW7, SW8, SW9: value Switch+Diode -> MX; footprint hb44:SMD_CherryMX_MidHeight_Choc_HotSwap+SOD123 -> hb44:SMD_CherryMX_MidHeight_HotSwap; moved to B.Cu
- SW15, SW5: value Switch+Diode -> MX; footprint hb44:SMD_CherryMX_MidHeight_Choc_HotSwap+SOD123 -> hb44:SMD_CherryMX_MidHeight_HotSwap
- SW16: footprint hb44:ec11 -> hb44:EC11
- U2: footprint Package_TO_SOT_SMD:SOT-363_SC-70-6_Handsoldering -> hb44:SMD_74AUP2G14_SOT-363; moved to B.Cu
- moved LED9 123.0 mm to (43.9, 54.0), turned to -90 degrees
- moved LED8 121.8 mm to (51.8, 44.4), turned to 180 degrees
- moved LED10 115.5 mm to (43.9, 72.1), turned to -90 degrees
- moved LED7 114.9 mm to (63.0, 34.9), turned to -90 degrees
- moved LED6 109.1 mm to (71.5, 32.4), turned to 180 degrees
- moved LED5 100.6 mm to (89.6, 30.1), turned to 180 degrees
- moved J2 98.7 mm to (101.8, 35.9), turned to -90 degrees
- moved LED4 95.5 mm to (110.7, 30.2), turned to 180 degrees
- moved LED3 91.8 mm to (118.1, 33.9), turned to 90 degrees
- moved LED11 91.2 mm to (43.9, 91.1), turned to -90 degrees
- moved LED12 88.1 mm to (52.4, 99.6)
- moved H1 81.1 mm to (113.4, 38.2)
- moved LED13 80.9 mm to (67.4, 104.3)
- moved Q1 62.2 mm to (119.2, 90.8), turned to -90 degrees
- moved D16 62.1 mm to (77.2, 41.2), turned to -90 degrees
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- renumbered D1 to D16
Connections:
- net /LED_VCC renamed LED_VCC
- C26 pad 1: Net-(C1-Pad1) -> R_LED_VCC
- C27 pad 1: Net-(C2-Pad1) -> R_LED_VCC
- J1 pad 1: HAP_1 -> +3V3
- J1 pad 2: SDA -> SDA/TX
- J1 pad 3: SCL -> SCL/RX
- J1 pad 4: SDA -> SDA/TX
- J1 pad 5: HAP_5 -> GND
- J2 pad 1: GND -> /RAW_BAT
- J2 pad 2: /RAW_BAT -> GND
- LCD1 pad 1: LCD_1 -> MOSI
- LCD1 pad 2: LCD_2 -> SCK
- LCD1 pad 3: VCC -> +3V3
- LCD1 pad 4: LCD_4 -> GND
- LCD1 pad 5: LCD_5 -> CS
- LED11 pad 1: Net-(LED11-Pad1) -> Net-(LED10-Pad3)
- LED11 pad 3: Net-(LED10-Pad1) -> Net-(LED11-Pad3)
- LED12 pad 1: Net-(LED12-Pad1) -> Net-(LED11-Pad3)
- LED12 pad 3: Net-(LED11-Pad1) -> Net-(LED12-Pad3)
- LED13 pad 1: Net-(LED13-Pad1) -> Net-(LED12-Pad3)
- LED13 pad 3: Net-(LED12-Pad1) -> Net-(LED13-Pad3)
- LED14 pad 1: Net-(LED14-Pad1) -> Net-(LED13-Pad3)
- LED14 pad 3: Net-(LED13-Pad1) -> Net-(LED14-Pad3)
- LED15 pad 1: Net-(LED15-Pad1) -> Net-(LED14-Pad3)
- LED15 pad 3: Net-(LED14-Pad1) -> unconnected-(LED15-Pad3)
- LED16 pad 1: Net-(LED16-Pad1) -> unconnected-(LED16-Pad1)
- LED16 pad 3: Net-(LED15-Pad1) -> Net-(LED16-Pad3)
- LED17 pad 1: Net-(LED17-Pad1) -> Net-(LED16-Pad3)
- LED22 pad 3: unconnected-(LED22-Pad3) -> Net-(LED22-Pad3)
- LED8 pad 3: Net-(LED16-Pad1) -> Net-(LED8-Pad3)
- LED9 pad 1: Net-(LED10-Pad3) -> Net-(LED8-Pad3)
- LED9 pad 3: Net-(LED17-Pad1) -> Net-(LED10-Pad1)
- Q1 pad 2: VCC -> +3V3
- R1 pad 1: VCC -> +3V3
- R2 pad 1: VCC -> +3V3
- R3 pad 2: Net-(C1-Pad1) -> Net-(C51-Pad1)
- R4 pad 2: Net-(C2-Pad1) -> Net-(C52-Pad1)
- SW1 pad 1: col1 -> col0
- SW10 pad 1: col5 -> col4
- SW11 pad 1: col1 -> col0
- SW12 pad 1: col2 -> col1
- SW13 pad 1: col3 -> col2
- SW14 pad 1: col4 -> col3
- SW15 pad 1: col5 -> col4
- SW16 pad S1: col2 -> col1
- SW17 pad 1: col3 -> col2
- SW18 pad 1: col4 -> col3
- SW19 pad 1: col5 -> col4
- SW2 pad 1: col2 -> col1
- SW20 pad 1: col1 -> col5
- SW3 pad 1: col3 -> col2
- SW4 pad 1: col4 -> col3
- SW5 pad 1: col5 -> col4
- SW6 pad 1: col1 -> col0
- SW7 pad 1: col2 -> col1
- SW8 pad 1: col3 -> col2
- SW9 pad 1: col4 -> col3
- U1 pad 10: col5 -> col4
- U1 pad 13: row3 -> col3
- U1 pad 14: row2 -> col2
- U1 pad 15: col3 -> col1
- U1 pad 16: col2 -> col0
- U1 pad 17: col1 -> row3
- U1 pad 18: col0 -> row2
- U1 pad 21: VCC -> +3V3
- U1 pad 23: GND -> GND1
- U1 pad 27: col4 -> col5
- U1 pad 6: MOSI -> SCK
- U1 pad 7: SCK -> MOSI
- U1 pad 8: SDA -> SCL/RX
- U1 pad 9: SCL -> SDA/TX
- U2 pad 1: Net-(C1-Pad1) -> Net-(C51-Pad1)
- U2 pad 3: Net-(C2-Pad1) -> Net-(C52-Pad1)
- U2 pad 5: VCC -> +3V3
Routing:
- net Net-(D5-Pad2): track 0.00 -> 146.1 mm
- net Net-(D21-Pad2): track 0.00 -> 133.3 mm
- net Net-(D10-Pad2): track 0.00 -> 121.0 mm
- net row2: track 4.54 -> 119.3 mm, vias 0 -> 4
- net Net-(D20-Pad2): track 0.00 -> 102.1 mm
- net Net-(D19-Pad2): track 0.00 -> 94.0 mm
- net row3: track 4.34 -> 97.4 mm, vias 0 -> 7
- net Net-(D15-Pad2): track 0.00 -> 89.6 mm
- net +3V3: track 0.00 -> 89.3 mm, vias 0 -> 4
- net Net-(D18-Pad2): track 0.00 -> 85.6 mm
- net Net-(D3-Pad2): track 8.52 -> 89.4 mm
- net rotS2: track 1.99 -> 80.7 mm, vias 0 -> 1
- net col0: track 0.00 -> 77.5 mm, vias 0 -> 4
- net Net-(D1-Pad2): track 8.52 -> 85.3 mm
- net row1: track 6.80 -> 83.2 mm, vias 0 -> 3
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- added copper zone on B.Cu, net GND3
- added copper zone on F.Cu, net LED_VCC
- added copper zone on F.Cu, net R_LED_VCC
- removed copper zone on F.Cu, net GND
Other:
- outline, holes or cut-outs redrawn
- board text added: "LED icon"
- board text added: "MCU/LCD icons"
- board text added: "battery icon"
- board text added: "encoder icon"
- board text added: "fingerprint icon"
- board text added: "haptic icon"
- board text added: "heartbreak"
- board text added: "magnet icon"
- board text added: "on/off!"
- board text added: "reset!"
- board text removed: "heartbreak - designed by drew"
