File: PCB/keyboard.kicad_sch (KiCad schematic)
At the start: 57 parts, among them J1 AudioJack4, J2 Conn_01x02, J3 Conn_01x05, SW1 Switch+Diode, SW10 Switch+Diode, SW11 Switch+Diode, SW12 Switch+Diode, SW13 Switch+Diode, SW14 Switch+Diode, SW15 Switch+Diode, SW16 Switch+Diode, SW17 Switch+Diode, SW18 RotaryEncoder_Switch, SW19 Switch+Diode, SW2 Switch+Diode, SW20 Switch+Diode, SW21 Switch+Diode, SW22 Switch+Diode, SW23 Switch+Diode, SW24 SW_PUSH, SW25 SW_DPDT_x2, SW3 Switch+Diode, SW4 Switch+Diode, SW5 Switch+Diode, SW6 Switch+Diode, SW7 Switch+Diode, SW8 Switch+Diode, SW9 Switch+Diode, U1 nice!nano

Commit message: folder structure
Parts:
- C1, C19, C2, C20: value 10n -> (none); footprint keyswitches:Cap_0603_Clean -> (none)
- D1: value (none) -> (none); footprint hb44:SMD_SOD123 -> (none)
- D2, D3, D4, D5, D6, D7, D8, D9: value WS2812B+Cap -> (none); footprint hb44:SMD_WS2812B+Cap0603 -> (none)
- J1: value AudioJack4 -> (none); footprint hb44:SMD_3.5mm_TRRS -> (none)
- J2: value Conn_01x02 -> (none); footprint hb44:TH_BatteryConn -> (none)
- J3: value Conn_01x05 -> (none); footprint hb44:Pimoroni Haptic Buzz DRV2605L Driver -> (none)
- JP1, JP2, JP3, JP4, JP5, JP6: value SolderJumper_3_Open -> (none); footprint keyswitches:jumperClean -> (none)
- LCD1: value nice!view -> (none); footprint hb44:nice!view -> (none)
- R1, R2, R3, R4, R5, R6, R7, R8: value 10k -> (none); footprint keyswitches:Res_1206_Clean -> (none)
- SW1, SW10, SW11, SW12, SW13, SW14, SW15, SW16, SW17, SW19, SW2, SW20, SW21, SW22, SW23, SW3, SW4, SW5, SW6, SW7, SW8, SW9: value Switch+Diode -> (none); footprint hb44:SMD_CherryMX_MidHeight_Choc_HotSwap+SOD123 -> (none)
- SW18: value RotaryEncoder_Switch -> (none); footprint keyswitches:ec11 -> (none)
- SW24: value SW_PUSH -> (none); footprint hb44:SMD_SW_PUSH -> (none)
- SW25: value SW_DPDT_x2 -> (none); footprint Button_Switch_SMD:SW_SPDT_PCM12 -> (none)
- U1: value nice!nano -> (none); footprint hb44:nice!nano -> (none)

Commit message: preliminary routing
Parts:
- C1, C19, C2, C20: value (none) -> 10n; footprint (none) -> hb44:Cap_0603_Clean
- D2, D3, D4, D5, D6, D7, D8, D9: value (none) -> WS2812B+Cap; footprint (none) -> hb44:SMD_WS2812B+Cap0603
- J1: value (none) -> AudioJack4; footprint (none) -> hb44:SMD_3.5mm_TRRS
- J2: value (none) -> Conn_01x02; footprint (none) -> hb44:TH_BatteryConn
- J3: value (none) -> Conn_01x05; footprint (none) -> hb44:Pimoroni Haptic Buzz DRV2605L Driver
- JP1, JP2, JP3, JP4, JP5, JP6: value (none) -> SolderJumper_3_Open; footprint (none) -> hb44:jumperClean
- LCD1: value (none) -> nice!view; footprint (none) -> hb44:nice!view
- R1, R2, R3, R4, R5, R6, R7, R8: value (none) -> 10k; footprint (none) -> hb44:Res_1206_Clean
- SW1, SW10, SW11, SW12, SW13, SW14, SW15, SW16, SW17, SW19, SW2, SW20, SW21, SW22, SW23, SW3, SW4, SW5, SW6, SW7, SW8, SW9: value (none) -> Switch+Diode; footprint (none) -> hb44:SMD_CherryMX_MidHeight_Choc_HotSwap+SOD123
- SW18: value (none) -> RotaryEncoder_Switch; footprint (none) -> hb44:ec11
- SW24: value (none) -> SW_PUSH; footprint (none) -> hb44:SMD_SW_PUSH
- SW25: value (none) -> SW_DPDT_x2; footprint (none) -> Button_Switch_SMD:SW_SPDT_PCM12
- U1: value (none) -> nice!nano; footprint (none) -> hb44:nice!nano

Commit message: wired compatible/breakaway
Parts:
- added Q1: (no value), symbol Device:Q_PMOS_GSD
- C1, C19, C2, C20: value 10n -> (none); footprint hb44:Cap_0603_Clean -> (none)
- D2, D3, D4, D5, D6, D7, D8, D9: value WS2812B+Cap -> (none); footprint hb44:SMD_WS2812B+Cap0603 -> (none)
- J1: value AudioJack4 -> (none); footprint hb44:SMD_3.5mm_TRRS -> (none)
- J2: value Conn_01x02 -> (none); footprint hb44:TH_BatteryConn -> (none)
- J3: value Conn_01x05 -> (none); footprint hb44:Pimoroni Haptic Buzz DRV2605L Driver -> (none)
- JP1, JP2, JP3, JP4, JP5, JP6: value SolderJumper_3_Open -> (none); footprint hb44:jumperClean -> (none)
- LCD1: value nice!view -> (none); footprint hb44:nice!view -> (none)
- R1, R2, R3, R4, R5, R6, R7, R8: value 10k -> (none); footprint hb44:Res_1206_Clean -> (none)
- SW1, SW10, SW11, SW12, SW13, SW14, SW15, SW16, SW17, SW19, SW2, SW20, SW21, SW22, SW23, SW3, SW4, SW5, SW6, SW7, SW8, SW9: value Switch+Diode -> (none); footprint hb44:SMD_CherryMX_MidHeight_Choc_HotSwap+SOD123 -> (none)
- SW18: value RotaryEncoder_Switch -> (none); footprint hb44:ec11 -> (none)
- SW24: value SW_PUSH -> (none); footprint hb44:SMD_SW_PUSH -> (none)
- SW25: value SW_DPDT_x2 -> (none); footprint Button_Switch_SMD:SW_SPDT_PCM12 -> (none)
- U1: value nice!nano -> (none); footprint hb44:nice!nano -> (none)

Commit message: curvy traces
Parts:
- removed C19, C20: (no value), symbol Device:C
- removed J1: (no value), symbol Connector:AudioJack4
- removed R5, R6, R7, R8: (no value), symbol Device:R
- added H1, H2, H3: (no value), symbol Mechanical:MountingHole
Connections:
- net CS: now also U1.5 (P0.17/H); no longer U1.2 (P0.08/H)
- net LED: now also Q1.1 (G), U1.2 (P0.08/H); no longer D2.4 (DIN), U1.1 (P0.06/H)
- net MOSI: now also U1.6 (P0.20/H); no longer U1.5 (P0.17/H)
- net SCK: now also U1.10 (P0.11/H); no longer U1.6 (P0.20/H)
- net SCL: now also U1.9 (P1.00/H); no longer U1.8 (P0.24/H)
- net SDA: now also U1.8 (P0.24/H); no longer U1.7 (P0.22/H)
- net VCC: now also Q1.3 (D); no longer D2.1, D3.1, D4.1, D5.1, D6.1, D7.1, D8.1, D9.1
- net col0: now also SW23.1 (COL); no longer SW22.1 (COL)
- net col1: now also SW22.1 (COL); no longer SW23.1 (COL)
- net col2: now also SW18.S1; no longer SW18.S2
- net col4: now also U1.25 (P1.01/L); no longer U1.14 (P0.10/L)
- net col5: now also U1.26 (P1.02/L); no longer U1.13 (P0.09/L)
- net rotA: now also U1.12 (P1.06/L); no longer U1.20 (P0.31/L)
- net rotB: now also U1.27 (P1.07/L); no longer U1.19 (P0.29/L)
- net row0: now also U1.20 (P0.31/L); no longer U1.9 (P1.00/H)
- net row1: now also U1.19 (P0.29/L); no longer U1.10 (P0.11/H)
- net row2: now also U1.14 (P0.10/L); no longer U1.11 (P1.04/L)
- net row3: now also U1.13 (P0.09/L); no longer U1.12 (P1.06/L)
- net LED_VCC: now reaches Q1.2 (S)
- net LED_VCC: now also D2.1, D3.1, D4.1, D5.1, D6.1, D7.1, D8.1, D9.1
- net RAW_BAT: now reaches J2.2 (Pin_2), SW25.3 (C)
- net rotS1 renamed rotS2
- net rotS2: now also SW18.S2; no longer SW18.S1
- new net ARGB: D2.4 (DIN), U1.1 (P0.06/H)
- no-connect marks 3 -> 4
Other:
- note added: "-..."
- note added: "-3x4mm press fit holes -Case pillars will slide into these"
- note added: "-Resets the microcontroller -Double tap to enter bootloader"
- note added: "Mounting Holes"
- note removed: "-Resets the microcontroller -Located at the top"
- note removed: "-Serial communication between boards -NOT hotswappable"
- note removed: "-some parts duplicated for an easy reversible footprint"
- note removed: "TRRS Jack"
- moved on the sheet: C1, C2, D2, D3, D4, D5, D6, D7, D8, D9, J2, J3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

Commit message: housekeeping
deleted unused files
Parts:
- C1, C2: value (none) -> 10n; footprint (none) -> hb44:SMD_Cap_0603
- D1: value (none) -> (none); footprint (none) -> hb44:SMD_SOD123
- D2, D3, D4, D5, D6, D7, D8, D9: value (none) -> WS2812B+Cap; footprint (none) -> hb44:SMD_WS2812B+Cap_0603
- H1, H2, H3: value (none) -> MountingHole; footprint (none) -> hb44:MountingHole_4mm
- J2: value (none) -> Conn_01x02; footprint (none) -> hb44:TH_BatteryConn
- J3: value (none) -> Conn_01x05; footprint (none) -> hb44:Pimoroni Haptic Buzz DRV2605L Driver
- JP1, JP2, JP3, JP4, JP5, JP6: value (none) -> SolderJumper_3_Open; footprint (none) -> hb44:SolderJumper
- LCD1: value (none) -> nice!view; footprint (none) -> hb44:nice!view
- Q1: value (none) -> Q_PMOS_GSD; footprint (none) -> hb44:SMD_P_MOSTFET_SOT-23
- R1, R2, R3, R4: value (none) -> 10k; footprint (none) -> hb44:SMD_Res_1206
- SW1, SW10, SW11, SW12, SW13, SW14, SW15, SW16, SW17, SW19, SW2, SW20, SW21, SW23, SW3, SW4, SW5, SW6, SW7, SW8, SW9: value (none) -> Switch+Diode; footprint (none) -> hb44:SMD_CherryMX_MidHeight_HotSwap+SOD123
- SW18: value (none) -> RotaryEncoder_Switch; footprint (none) -> hb44:EC11
- SW24: value (none) -> SW_PUSH; footprint (none) -> hb44:SMD_SW_SPST_B3U-3000P-B
- SW25: value (none) -> SW_DPDT_x2; footprint (none) -> hb44:SMD_SW_SPDT_PCM12
- U1: value (none) -> nice!nano; footprint (none) -> hb44:nice!nano

Commit message: working 44
Parts:
- added J?: Conn_01x05, hb44:Pimoroni Haptic Buzz DRV2605L Driver, symbol Connector_Generic:Conn_01x04
- added R5: 200, symbol Device:R
- added R6: 200k, symbol Device:R
- H1, H2, H3: footprint hb44:MountingHole_4mm -> hb44:MountingHole_4.1mm
- SW18: footprint hb44:EC11 -> hb44:ec11
- SW22: value (none) -> Switch+Diode; footprint (none) -> hb44:SMD_CherryMX_MidHeight_HotSwap+SOD123
Connections:
- net ARGB: now also U1.10 (P0.11/H); no longer U1.1 (P0.06/H)
- net GND: now also J?.4 (Pin_4), R6.2
- net LED: now also U1.11 (P1.04/L), R5.1, R6.1; no longer Q1.1 (G), U1.2 (P0.08/H)
- net LED_VCC: now also Q1.3 (D); no longer Q1.2 (S)
- net SCK: now also U1.7 (P0.22/H); no longer U1.10 (P0.11/H)
- net VCC: now also Q1.2 (S), J?.1 (Pin_1); no longer Q1.3 (D)
- new net: Q1.1 (G), R5.2
- new net RX: J?.2 (Pin_2), U1.2 (P0.08/H)
- new net TX: J?.3 (Pin_3), U1.1 (P0.06/H)
- no-connect marks 4 -> 2
Other:
- note added: "-3x4.1mm press fit holes -Case pillars will slide into these"
- note added: "-Individually addressible RGB LEDs -Decoupled with 0.1uF capacitors -Toggled with mosfet for power savings"
- note added: "-USB C Breakout with 21 GPIO pins -Uses BLE to work with sister half"
- note added: "-adafruit 4750 -interfaces over UART"
- note added: "Fingerprint Reader"
- note removed: "-3x4mm press fit holes -Case pillars will slide into these"
- note removed: "-Individually addressible RGB LEDs -Decoupled with 0.1uF capacitors"
- note removed: "-USB C Pro Micro with 18 GPIO pins -Uses serial communication to work with sister half"
- moved on the sheet: D2, D3, D4, D5, D6, D7, D8, D9, J3, JP5, JP6, Q1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

Commit message: reversible WIP
Parts:
- removed SW1, SW7: Switch+Diode, hb44:SMD_CherryMX_MidHeight_HotSwap+SOD123, symbol hb44:Switch+Diode
- added LED10, LED11, LED12, LED13, LED14, LED15, LED16, LED17, LED18, LED19, LED20, LED21, LED22, LED9: 0.1u, keyswitches:ledClean, symbol hb44:SK6812+Cap
- added U2: 74AUP2G14, Package_TO_SOT_SMD:SOT-363_SC-70-6_Handsoldering, symbol hb44:74AUP2G14
- C1, C2: value 10n -> 0.1u
- J1: renamed from J?; now left out of the parts list
- LED1: renamed from D2; value WS2812B+Cap -> 0.1u; footprint hb44:SMD_WS2812B+Cap_0603 -> keyswitches:ledClean; symbol hb44:WS2812B+Cap -> hb44:SK6812+Cap
- LED2: renamed from D3; value WS2812B+Cap -> 0.1u; footprint hb44:SMD_WS2812B+Cap_0603 -> keyswitches:ledClean; symbol hb44:WS2812B+Cap -> hb44:SK6812+Cap
- LED3: renamed from D4; value WS2812B+Cap -> 0.1u; footprint hb44:SMD_WS2812B+Cap_0603 -> keyswitches:ledClean; symbol hb44:WS2812B+Cap -> hb44:SK6812+Cap
- LED4: renamed from D5; value WS2812B+Cap -> 0.1u; footprint hb44:SMD_WS2812B+Cap_0603 -> keyswitches:ledClean; symbol hb44:WS2812B+Cap -> hb44:SK6812+Cap
- LED5: renamed from D6; value WS2812B+Cap -> 0.1u; footprint hb44:SMD_WS2812B+Cap_0603 -> keyswitches:ledClean; symbol hb44:WS2812B+Cap -> hb44:SK6812+Cap
- LED6: renamed from D7; value WS2812B+Cap -> 0.1u; footprint hb44:SMD_WS2812B+Cap_0603 -> keyswitches:ledClean; symbol hb44:WS2812B+Cap -> hb44:SK6812+Cap
- LED7: renamed from D8; value WS2812B+Cap -> 0.1u; footprint hb44:SMD_WS2812B+Cap_0603 -> keyswitches:ledClean; symbol hb44:WS2812B+Cap -> hb44:SK6812+Cap
- LED8: renamed from D9; value WS2812B+Cap -> 0.1u; footprint hb44:SMD_WS2812B+Cap_0603 -> keyswitches:ledClean; symbol hb44:WS2812B+Cap -> hb44:SK6812+Cap
- Q1: footprint hb44:SMD_P_MOSTFET_SOT-23 -> hb44:SMD_P_MOSFET_SOT-23
- R1: value 10k -> (none); footprint hb44:SMD_Res_1206 -> (none)
- R5, R6: footprint (none) -> hb44:SMD_Res_1206
- renumbered SW2 to SW1, SW12 to SW10, SW13 to SW11, SW14 to SW12, SW15 to SW13, SW16 to SW14, SW17 to SW15, SW18 to SW16, SW19 to SW17, SW20 to SW18, SW21 to SW19, SW3 to SW2, SW22 to SW20, SW23 to SW21, SW4 to SW3, SW5 to SW4, SW6 to SW5, SW8 to SW6, SW9 to SW7, SW10 to SW8, SW11 to SW9
Connections:
- net ARGB: now also LED1.1 (DIN), U1.1 (P0.06/H); no longer LED1.4 (DIN), U1.10 (P0.11/H)
- net GND: now also LED1.4, LED2.4, LED3.4, LED4.4, LED5.4, LED6.4, LED7.4, LED8.4, LED10.4, LED11.4, LED12.4, LED13.4, LED14.4, LED15.4, LED16.4, LED17.4, LED18.4, LED19.4, LED20.4, LED21.4, LED22.4, LED9.4, U2.2 (GND); no longer LED1.3, LED2.3, LED3.3, LED4.3, LED5.3, LED6.3, LED7.3, LED8.3
- net LED: now also U1.2 (P0.08/H); no longer U1.11 (P1.04/L)
- net LED_VCC: now also LED1.2, LED2.2, LED3.2, LED4.2, LED5.2, LED6.2, LED7.2, LED8.2, LED10.2, LED11.2, LED12.2, LED13.2, LED14.2, LED15.2, LED16.2, LED17.2, LED18.2, LED19.2, LED20.2, LED21.2, LED22.2, LED9.2; no longer LED1.1, LED2.1, LED3.1, LED4.1, LED5.1, LED6.1, LED7.1, LED8.1
- net SCL: now also J1.3 (Pin_3)
- net SDA: now also J1.2 (Pin_2)
- net VCC: now also U2.5 (VCC)
- net col4: now also U1.27 (P1.07/L); no longer U1.25 (P1.01/L)
- net col5: now also U1.10 (P0.11/H); no longer U1.26 (P1.02/L)
- net rotA: now also U2.6; no longer C1.1, R3.2
- net rotB: now also U1.11 (P1.04/L), U2.4; no longer C2.1, R4.2, U1.27 (P1.07/L)
- removed net RX: J1.2 (Pin_2), U1.2 (P0.08/H)
- removed net TX: J1.3 (Pin_3), U1.1 (P0.06/H)
- new net: LED17.1 (DIN), LED9.3 (DOUT)
- new net: LED17.3 (DOUT), LED18.1 (DIN)
- new net: LED11.1 (DIN), LED12.3 (DOUT)
- new net: LED10.1 (DIN), LED11.3 (DOUT)
- new net: LED18.3 (DOUT), LED19.1 (DIN)
- new net: LED19.3 (DOUT), LED20.1 (DIN)
- new net: LED7.3 (DOUT), LED8.1 (DIN)
- new net: LED16.1 (DIN), LED8.3 (DOUT)
- new net: LED21.3 (DOUT), LED22.1 (DIN)
- new net: LED15.1 (DIN), LED16.3 (DOUT)
- new net: LED14.1 (DIN), LED15.3 (DOUT)
- new net: LED20.3 (DOUT), LED21.1 (DIN)
- new net: LED6.3 (DOUT), LED7.1 (DIN)
- new net: LED13.1 (DIN), LED14.3 (DOUT)
- new net: C1.1, R3.2, U2.1
- new net: C2.1, R4.2, U2.3
- new net: LED1.3 (DOUT), LED2.1 (DIN)
- new net: LED2.3 (DOUT), LED3.1 (DIN)
- new net: LED12.1 (DIN), LED13.3 (DOUT)
- new net: LED3.3 (DOUT), LED4.1 (DIN)
- new net: LED5.3 (DOUT), LED6.1 (DIN)
- new net: LED10.3 (DOUT), LED9.1 (DIN)
- new net: LED4.3 (DOUT), LED5.1 (DIN)
- no-connect marks 2 -> 4
Other:
- note added: "-22 Individually addressible RGB LEDs -Decoupled with 0.1uF capacitors -Toggled with mosfet for power savings"
- note added: "-Low pass filter and Schmitt trigger debounce -Also functions as a switch"
- note added: "-adafruit 4750 and uses UART -mutually exclusive with haptic"
- note removed: "-Individually addressible RGB LEDs -Decoupled with 0.1uF capacitors -Toggled with mosfet for power savings"
- note removed: "-Uses an RC filter for debouncing -Also functions as a switch"
- note removed: "-adafruit 4750 -interfaces over UART"
- moved on the sheet: C1, C2, LED1, LED2, LED3, LED4, LED5, LED6, LED7, LED8, Q1, R1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

Commit message: vertical
Parts:
- removed J1: Conn_01x05, hb44:Pimoroni Haptic Buzz DRV2605L Driver, symbol Connector_Generic:Conn_01x04
- removed JP1, JP2, JP3, JP4, JP5, JP6: SolderJumper_3_Open, hb44:SolderJumper, symbol Jumper:SolderJumper_3_Open
- removed LED14, LED15, LED16, LED22, LED6, LED7, LED8: 0.1u, keyswitches:ledClean, symbol hb44:SK6812+Cap
- removed SW24: SW_PUSH, hb44:SMD_SW_SPST_B3U-3000P-B, symbol kbd:SW_PUSH
- removed SW25: SW_DPDT_x2, hb44:SMD_SW_SPDT_PCM12, symbol Switch:SW_DPDT_x2
- added C10, C11, C12, C13, C14, C15, C16, C17, C18, C19, C20, C21, C22, C23, C24, C25, C26, C27, C28, C29, C3, C30, C31, C32, C33, C34, C35, C36, C37, C38, C39, C4, C40, C41, C42, C43, C44, C45, C46, C47, C48, C49, C5, C50, C51, C52, C53, C54, C6, C7, C8, C9: 0.1u, hb44:SMD_Cap_0603, symbol Device:C
- added D10, D11, D12, D13, D14, D15, D16, D17, D18, D19, D2, D20, D21, D22, D23, D24, D25, D26, D27, D28, D29, D3, D30, D31, D32, D33, D34, D35, D36, D37, D38, D39, D4, D40, D41, D42, D5, D6, D7, D8, D9: (no value), hb44:SMD_SOD123, symbol Device:D_Small
- added H10, H11, H12, H13, H14, H15, H16, H4, H5, H6, H7, H8, H9: MountingHole, hb44:MountingHole_4mm, symbol Mechanical:MountingHole
- added J1: Conn_01x05, hb44:Pimoroni Haptic Buzz, symbol Connector_Generic:Conn_01x05
- added J1X1, J3X1: Conn_01x05, hb44:Pimoroni Haptic Buzz, symbol Connector_Generic:Conn_01x04
- added J4: Conn_01x02, hb44:TH_BatteryConn, symbol Connector_Generic:Conn_01x02
- added LCD2: nice!view, hb44:nice!view, symbol hb44:nice!view
- added LED16, LED17, LED18, LED19, LED20, LED21, LED22, LED23, LED24, LED25, LED26, LED27, LED28, LED29, LED30, LED31, LED32, LED33, LED34, LED35, LED36, LED37, LED38, LED39, LED40, LED41, LED42, LED43, LED44, LED45, LED46, LED47, LED48, LED49, LED50: SK6812, hb44:SK6812-SIDE, symbol hb44:SK6812
- added Q2: Q_PMOS_GSD, hb44:SMD_P_MOSFET_SOT-23, symbol Device:Q_PMOS_GSD
- added R10, R7, R8, R9: 10k, hb44:SMD_Res_1206, symbol Device:R
- added R11: 200, hb44:SMD_Res_1206, symbol Device:R
- added R12: 200k, hb44:SMD_Res_1206, symbol Device:R
- added SW22, SW23, SW24, SW25, SW26, SW27, SW28, SW29, SW30, SW31, SW32, SW33, SW34, SW35, SW36, SW38, SW39, SW40, SW41, SW42: MX, hb44:SMD_CherryMX_MidHeight_HotSwap, symbol hb44:Switch
- added SW37: RotaryEncoder_Switch, hb44:EC11, symbol Device:RotaryEncoder_Switch
- added SW43, SW45: SW_DPDT_x2, hb44:SMD_SW_SPDT_PCM12, symbol Switch:SW_DPDT_x2
- added SW44, SW46: SW_PUSH, hb44:SMD_SW_SPST_B3U-3000P-B, symbol kbd:SW_PUSH
- added U3: nice!nano, hb44:nice!nano, symbol hb44:nice!nano
- added U4: 74AUP2G14, hb44:SMD_74AUP2G14_SOT-363, symbol hb44:74AUP2G14
- H1, H2, H3: footprint hb44:MountingHole_4.1mm -> hb44:MountingHole_4mm
- J3: footprint hb44:Pimoroni Haptic Buzz DRV2605L Driver -> hb44:Pimoroni Haptic Buzz
- LED1, LED2, LED3, LED4, LED5: value 0.1u -> SK6812; footprint keyswitches:ledClean -> hb44:SK6812-SIDE; symbol hb44:SK6812+Cap -> hb44:SK6812
- LED10: renamed from LED9; value 0.1u -> SK6812; footprint keyswitches:ledClean -> hb44:SK6812-SIDE; symbol hb44:SK6812+Cap -> hb44:SK6812
- LED11: renamed from LED17; value 0.1u -> SK6812; footprint keyswitches:ledClean -> hb44:SK6812-SIDE; symbol hb44:SK6812+Cap -> hb44:SK6812
- LED12: renamed from LED18; value 0.1u -> SK6812; footprint keyswitches:ledClean -> hb44:SK6812-SIDE; symbol hb44:SK6812+Cap -> hb44:SK6812
- LED13: renamed from LED19; value 0.1u -> SK6812; footprint keyswitches:ledClean -> hb44:SK6812-SIDE; symbol hb44:SK6812+Cap -> hb44:SK6812
- LED14: renamed from LED20; value 0.1u -> SK6812; footprint keyswitches:ledClean -> hb44:SK6812-SIDE; symbol hb44:SK6812+Cap -> hb44:SK6812
- LED15: renamed from LED21; value 0.1u -> SK6812; footprint keyswitches:ledClean -> hb44:SK6812-SIDE; symbol hb44:SK6812+Cap -> hb44:SK6812
- LED6: renamed from LED13; value 0.1u -> SK6812; footprint keyswitches:ledClean -> hb44:SK6812-SIDE; symbol hb44:SK6812+Cap -> hb44:SK6812
- LED7: renamed from LED12; value 0.1u -> SK6812; footprint keyswitches:ledClean -> hb44:SK6812-SIDE; symbol hb44:SK6812+Cap -> hb44:SK6812
- LED8: renamed from LED11; value 0.1u -> SK6812; footprint keyswitches:ledClean -> hb44:SK6812-SIDE; symbol hb44:SK6812+Cap -> hb44:SK6812
- LED9: renamed from LED10; value 0.1u -> SK6812; footprint keyswitches:ledClean -> hb44:SK6812-SIDE; symbol hb44:SK6812+Cap -> hb44:SK6812
- R1: value (none) -> 10k; footprint (none) -> hb44:SMD_Res_1206
- SW1, SW10, SW11, SW12, SW13, SW14, SW15, SW17, SW18, SW19, SW2, SW20, SW21, SW3, SW4, SW5, SW6, SW7, SW8, SW9: value Switch+Diode -> MX; footprint hb44:SMD_CherryMX_MidHeight_HotSwap+SOD123 -> hb44:SMD_CherryMX_MidHeight_HotSwap; symbol hb44:Switch+Diode -> hb44:Switch
- SW16: footprint hb44:ec11 -> hb44:EC11
- U2: footprint Package_TO_SOT_SMD:SOT-363_SC-70-6_Handsoldering -> hb44:SMD_74AUP2G14_SOT-363
Connections:
- net HAP_5 is gone; now on net GND: J3.5 (Pin_5)
- net LCD_1 is gone; now on net MOSI: LCD1.1 (MOSI)
- net LCD_2 is gone; now on net SCK: LCD1.2 (SCK)
- net LCD_4 is gone; now on net GND: LCD1.4 (GND)
- net LCD_5 is gone; now on net CS: LCD1.5 (CS)
- net VCC is gone; now on net +3V3: LCD1.3 (VCC), Q1.2 (S), R1.1, R2.1, U1.21 (3.3V), U2.5 (VCC)
- net GND: now also J2.2 (Pin_2), C10.1, C11.2, C12.2, C13.2, C14.2, C15.2, C16.1, C17.1, C18.1, C19.1, C20.1, C21.2, C22.2, C23.2, C24.2, C26.2, C27.2, C28.2, C29.2, C3.2, C30.2, C31.1, C32.1, C33.1, C34.1, C35.1, C36.2, C37.2, C38.2, C39.2, C4.2, C40.2, C46.2, C47.2, C48.2, C49.2, C5.2, C51.2, C52.2, C53.2, C54.2, C6.1, C7.1, C8.1, C9.1, J1.5 (Pin_5), J1X1.4 (Pin_4), J3X1.4 (Pin_4), J4.2 (Pin_2), LCD2.4 (GND), LED16.4 (VSS), LED17.4 (VSS), LED18.4 (VSS), LED19.4 (VSS), LED20.4 (VSS), LED21.4 (VSS), LED22.4 (VSS), LED23.4 (VSS), LED24.4 (VSS), LED26.4 (VSS), LED27.4 (VSS), LED28.4 (VSS), LED29.4 (VSS), LED30.4 (VSS), LED31.4 (VSS), LED32.4 (VSS), LED33.4 (VSS), LED34.4 (VSS), LED35.4 (VSS), LED36.4 (VSS), LED37.4 (VSS), LED38.4 (VSS), LED39.4 (VSS), LED40.4 (VSS), LED41.4 (VSS), LED42.4 (VSS), LED43.4 (VSS), LED44.4 (VSS), LED45.4 (VSS), LED46.4 (VSS), LED47.4 (VSS), LED48.4 (VSS), LED49.4 (VSS), R12.2, SW37.C, SW44.2, SW46.2, U3.23 (GND), U4.2 (GND); no longer J2.1 (Pin_1), U1.23 (GND)
- net LED_VCC: now also C1.1, C2.1, C10.2, C11.1, C12.1, C13.1, C14.1, C15.1, C16.2, C17.2, C18.2, C19.2, C20.2, C21.1, C22.1, C23.1, C24.1, C25.1, C3.1, C4.1, C5.1, C6.2, C7.2, C8.2, C9.2, LED16.2 (VDD), LED17.2 (VDD), LED18.2 (VDD), LED19.2 (VDD), LED20.2 (VDD), LED21.2 (VDD), LED22.2 (VDD), LED23.2 (VDD), LED24.2 (VDD), LED25.2 (VDD)
- net MOSI: now also U1.7 (P0.22/H); no longer U1.6 (P0.20/H)
- net RAW: now also SW43.2 (B)
- net RAW_BAT: now also J2.1 (Pin_1), SW43.1 (A); no longer J2.2 (Pin_2)
- net RESET: now also SW44.1
- net SCK: now also U1.6 (P0.20/H); no longer U1.7 (P0.22/H)
- net col0: now also SW1.1 (COL), SW11.1 (COL), SW6.1 (COL), U1.16 (P1.13/L); no longer U1.18 (P0.02/L)
- net col1: now also SW12.1 (COL), SW16.S1, SW2.1 (COL), SW7.1 (COL), U1.15 (P1.11/L); no longer SW1.1 (COL), SW11.1 (COL), SW20.1 (COL), SW6.1 (COL), U1.17 (P1.15/L)
- net col2: now also SW13.1 (COL), SW17.1 (COL), SW3.1 (COL), SW8.1 (COL), U1.14 (P0.10/L); no longer SW12.1 (COL), SW16.S1, SW2.1 (COL), SW7.1 (COL), U1.16 (P1.13/L)
- net col3: now also SW14.1 (COL), SW18.1 (COL), SW4.1 (COL), SW9.1 (COL), U1.13 (P0.09/L); no longer SW13.1 (COL), SW17.1 (COL), SW3.1 (COL), SW8.1 (COL), U1.15 (P1.11/L)
- net col4: now also SW10.1 (COL), SW15.1 (COL), SW19.1 (COL), SW5.1 (COL), U1.10 (P0.11/H); no longer SW14.1 (COL), SW18.1 (COL), SW4.1 (COL), SW9.1 (COL), U1.27 (P1.07/L)
- net col5: now also SW20.1 (COL), U1.27 (P1.07/L); no longer SW10.1 (COL), SW15.1 (COL), SW19.1 (COL), SW5.1 (COL), U1.10 (P0.11/H)
- net rotS2: now also D16.2 (A); no longer D1.2 (A)
- net row0: now also D1.1 (K), D2.1 (K), D3.1 (K), D4.1 (K), D5.1 (K); no longer SW1.3, SW2.3, SW3.3, SW4.3, SW5.3
- net row1: now also D10.1 (K), D6.1 (K), D7.1 (K), D8.1 (K), D9.1 (K); no longer SW10.3, SW6.3, SW7.3, SW8.3, SW9.3
- net row2: now also U1.18 (P0.02/L), D11.1 (K), D12.1 (K), D13.1 (K), D14.1 (K), D15.1 (K); no longer SW11.3, SW12.3, SW13.3, SW14.3, SW15.3, U1.14 (P0.10/L)
- net row3: now also U1.17 (P1.15/L), D16.1 (K), D17.1 (K), D18.1 (K), D19.1 (K), D20.1 (K), D21.1 (K); no longer D1.1 (K), SW17.3, SW18.3, SW19.3, SW20.3, SW21.3, U1.13 (P0.09/L)
- net at SW17.2 (ROW): now also D17.2 (A)
- net at SW4.2 (ROW): now also D4.2 (A)
- net at SW1.2 (ROW): now also D1.2 (A)
- net at SW3.2 (ROW): now also D3.2 (A)
- net at SW15.2 (ROW): now also D15.2 (A)
- net at SW14.2 (ROW): now also D14.2 (A)
- net at LED6.1 (DIN): now also LED5.3 (DOUT)
- net at R3.2, U2.1: now also C51.1; no longer C1.1
- net at R4.2, U2.3: now also C52.1; no longer C2.1
- net at SW18.2 (ROW): now also D18.2 (A)
- net at SW21.2 (ROW): now also D21.2 (A)
- net at SW9.2 (ROW): now also D9.2 (A)
- net at SW19.2 (ROW): now also D19.2 (A)
- net at SW12.2 (ROW): now also D12.2 (A)
- net at SW5.2 (ROW): now also D5.2 (A)
- net at SW20.2 (ROW): now also D20.2 (A)
- net at SW11.2 (ROW): now also D11.2 (A)
- net at SW7.2 (ROW): now also D7.2 (A)
- net at SW13.2 (ROW): now also D13.2 (A)
- net at SW2.2 (ROW): now also D2.2 (A)
- net at SW6.2 (ROW): now also D6.2 (A)
- net at SW8.2 (ROW): now also D8.2 (A)
- net at SW10.2 (ROW): now also D10.2 (A)
- net HAP_1 renamed +3V3
- net +3V3: now also J1.1 (Pin_1), J1X1.1 (Pin_1), J3X1.1 (Pin_1), LCD2.3 (VCC), Q2.2 (S), R7.1, R8.1, U3.21 (3.3V), U4.5 (VCC)
- net SCL renamed R_SCL/RX
- net R_SCL/RX: now also J3X1.3 (Pin_3), U3.8 (P0.24/H); no longer U1.9 (P1.00/H)
- net SDA renamed R_SDA/TX
- net R_SDA/TX: now also J3X1.2 (Pin_2), U3.9 (P1.00/H); no longer U1.8 (P0.24/H)
- new net: LED38.3 (DOUT), LED39.1 (DIN)
- new net: LED39.3 (DOUT), LED40.1 (DIN)
- new net: D26.2 (A), SW26.2 (ROW)
- new net: LED45.3 (DOUT), LED46.1 (DIN)
- new net: D23.2 (A), SW23.2 (ROW)
- new net: LED35.3 (DOUT), LED36.1 (DIN)
- new net: LED36.3 (DOUT), LED37.1 (DIN)
- new net: D24.2 (A), SW24.2 (ROW)
- new net: D40.2 (A), SW40.2 (ROW)
- new net: D29.2 (A), SW29.2 (ROW)
- new net: D33.2 (A), SW33.2 (ROW)
- new net: LED33.3 (DOUT), LED34.1 (DIN)
- new net: LED34.3 (DOUT), LED35.1 (DIN)
- new net: R7.2, R9.1, SW37.A
- new net: C53.1, R9.2, U4.1
- new net: D28.2 (A), SW28.2 (ROW)
- new net: LED32.3 (DOUT), LED33.1 (DIN)
- new net: D39.2 (A), SW39.2 (ROW)
- new net: LED28.3 (DOUT), LED29.1 (DIN)
- new net: LED29.3 (DOUT), LED30.1 (DIN)
- new net: D30.2 (A), SW30.2 (ROW)
- new net: LED16.3 (DOUT), LED17.1 (DIN)
- new net: LED17.3 (DOUT), LED18.1 (DIN)
- new net: LED47.3 (DOUT), LED48.1 (DIN)
- new net: LED48.3 (DOUT), LED49.1 (DIN)
- new net: R10.1, R8.2, SW37.B
- new net: C54.1, R10.2, U4.3
- new net: D32.2 (A), SW32.2 (ROW)
- new net: LED46.3 (DOUT), LED47.1 (DIN)
- new net: LED27.3 (DOUT), LED28.1 (DIN)
- new net: D41.2 (A), SW41.2 (ROW)
- new net: LED19.3 (DOUT), LED20.1 (DIN)
- new net: LED20.3 (DOUT), LED21.1 (DIN)
- new net: Q2.1 (G), R11.2
- new net: D27.2 (A), SW27.2 (ROW)
- new net: LED37.3 (DOUT), LED38.1 (DIN)
- new net: LED23.3 (DOUT), LED24.1 (DIN)
- new net: LED24.3 (DOUT), LED25.1 (DIN)
- new net: D35.2 (A), SW35.2 (ROW)
- new net: LED26.3 (DOUT), LED27.1 (DIN)
- new net: D36.2 (A), SW36.2 (ROW)
- new net: LED21.3 (DOUT), LED22.1 (DIN)
- new net: LED22.3 (DOUT), LED23.1 (DIN)
- new net: D34.2 (A), SW34.2 (ROW)
- new net: LED49.3 (DOUT), LED50.1 (DIN)
- new net: LED31.3 (DOUT), LED32.1 (DIN)
- new net: D31.2 (A), SW31.2 (ROW)
- new net: D42.2 (A), SW42.2 (ROW)
- new net: D22.2 (A), SW22.2 (ROW)
- new net: D38.2 (A), SW38.2 (ROW)
- new net: LED18.3 (DOUT), LED19.1 (DIN)
- new net: D25.2 (A), SW25.2 (ROW)
- new net: LED30.3 (DOUT), LED31.1 (DIN)
- new net GND1: C25.2, LED25.4 (VSS), U1.23 (GND)
- new net GND3: C50.2, LED50.4 (VSS), U3.3 (GND), U3.4 (GND)
- new net R_ARGB: LED26.1 (DIN), U3.1 (P0.06/H)
- new net R_CS: LCD2.5 (CS), U3.5 (P0.17/H)
- new net R_LED: R11.1, R12.1, U3.2 (P0.08/H)
- new net R_LED_VCC: C26.1, C27.1, C28.1, C29.1, C30.1, C31.2, C32.2, C33.2, C34.2, C35.2, C36.1, C37.1, C38.1, C39.1, C40.1, C46.1, C47.1, C48.1, C49.1, C50.1, LED26.2 (VDD), LED27.2 (VDD), LED28.2 (VDD), LED29.2 (VDD), LED30.2 (VDD), LED31.2 (VDD), LED32.2 (VDD), LED33.2 (VDD), LED34.2 (VDD), LED35.2 (VDD), LED36.2 (VDD), LED37.2 (VDD), LED38.2 (VDD), LED39.2 (VDD), LED40.2 (VDD), LED41.2 (VDD), LED42.2 (VDD), LED43.2 (VDD), LED44.2 (VDD), LED45.2 (VDD), LED46.2 (VDD), LED47.2 (VDD), LED48.2 (VDD), LED49.2 (VDD), LED50.2 (VDD), Q2.3 (D)
- new net R_MOSI: LCD2.1 (MOSI), U3.7 (P0.22/H)
- new net R_RAW: SW45.2 (B), U3.24 (BAT+)
- new net R_RAW_BAT: J4.1 (Pin_1), SW45.1 (A)
- new net R_RESET: SW46.1, U3.22 (RESET)
- new net R_SCK: LCD2.2 (SCK), U3.6 (P0.20/H)
- new net R_col0: SW22.1 (COL), SW27.1 (COL), SW32.1 (COL), SW42.1 (COL), U3.16 (P1.13/L)
- new net R_col1: SW23.1 (COL), SW28.1 (COL), SW33.1 (COL), SW37.S1, U3.15 (P1.11/L)
- new net R_col2: SW24.1 (COL), SW29.1 (COL), SW34.1 (COL), SW38.1 (COL), U3.14 (P0.10/L)
- new net R_col3: SW25.1 (COL), SW30.1 (COL), SW35.1 (COL), SW39.1 (COL), U3.13 (P0.09/L)
- new net R_col4: SW26.1 (COL), SW31.1 (COL), SW36.1 (COL), SW40.1 (COL), U3.10 (P0.11/H)
- new net R_col5: SW41.1 (COL), U3.27 (P1.07/L)
- new net R_rotA: U3.12 (P1.06/L), U4.6
- new net R_rotB: U3.11 (P1.04/L), U4.4
- new net R_rotS2: D37.2 (A), SW37.S2
- new net R_row0: D22.1 (K), D23.1 (K), D24.1 (K), D25.1 (K), D26.1 (K), U3.20 (P0.31/L)
- new net R_row1: D27.1 (K), D28.1 (K), D29.1 (K), D30.1 (K), D31.1 (K), U3.19 (P0.29/L)
- new net R_row2: D32.1 (K), D33.1 (K), D34.1 (K), D35.1 (K), D36.1 (K), U3.18 (P0.02/L)
- new net R_row3: D37.1 (K), D38.1 (K), D39.1 (K), D40.1 (K), D41.1 (K), D42.1 (K), U3.17 (P1.15/L)
- new net SCL/RX: J1.3 (Pin_3), J1X1.3 (Pin_3), U1.8 (P0.24/H)
- new net SDA/TX: J1.2 (Pin_2), J1.4 (Pin_4), J1X1.2 (Pin_2), U1.9 (P1.00/H)
- no-connect marks 4 -> 8
Other:
- note added: "-4mm clearance holes -Allows mating magnets"
- note added: "-4x6 matrix, 21 switches -Hotswap MX footprint"
- note added: "-Low pass filter and Schmitt trigger d -Also functions as a switch"
- note added: "Battery + Switch"
- note added: "L"
- note added: "Mounting"
- note added: "R"
- note removed: "-..."
- note removed: "-3x4.1mm press fit holes -Case pillars will slide into these"
- note removed: "-4x6 matrix, 23 switches -Hotswap MX/Choc footprint"
- note removed: "-Low pass filter and Schmitt trigger debounce -Also functions as a switch"
- note removed: "Battery Switch"
- note removed: "Mounting Holes"
- note removed: "Notes:"
- title: hb44 -> heartbreak
- moved on the sheet: Q1, R5, R6, U1
