File: PCB/keyboard.kicad_sch (KiCad schematic)
At the start: 234 parts, among them J1 Conn_01x05, J1X1 Conn_01x05, J2 Conn_01x02, J3 Conn_01x05, J3X1 Conn_01x05, J4 Conn_01x02, Q1 Q_PMOS_GSD, Q2 Q_PMOS_GSD, SW1 MX, SW10 MX, SW11 MX, SW12 MX, SW13 MX, SW14 MX, SW15 MX, SW16 RotaryEncoder_Switch, SW17 MX, SW18 MX, SW19 MX, SW2 MX, SW20 MX, SW21 MX, SW22 MX, SW23 MX, SW24 MX, SW25 MX, SW26 MX, SW27 MX, SW28 MX, SW29 MX, SW3 MX, SW30 MX, SW31 MX, SW32 MX, SW33 MX, SW34 MX, SW35 MX, SW36 MX, SW37 RotaryEncoder_Switch, SW38 MX, SW39 MX, SW4 MX, SW40 MX, SW41 MX, SW42 MX, SW43 SW_DPDT_x2, SW44 SW_PUSH, SW45 SW_DPDT_x2, SW46 SW_PUSH, SW5 MX, SW6 MX, SW7 MX, SW8 MX, SW9 MX, U1 nice!nano, U2 74AUP2G14, U3 nice!nano, U4 74AUP2G14

Commit message: production
Parts:
- removed C14, C15, C16, C17, C18, C19, C20, C21, C22, C23, C24, C25, C26, C27, C28, C29, C30, C31, C32, C33, C34, C35, C36, C37, C38, C39, C40, C41, C42, C43, C44, C45, C46, C47, C48, C49, C50, C53, C54: 0.1u, hb44:SMD_Cap_0603, symbol Device:C
- removed D22, D23, D24, D25, D26, D27, D28, D29, D30, D31, D32, D33, D34, D35, D36, D37, D38, D39, D40, D41, D42: (no value), hb44:SMD_SOD123, symbol Device:D_Small
- removed H10, H11, H12, H13, H14, H15, H16, H9: MountingHole, hb44:MountingHole_4mm, symbol Mechanical:MountingHole
- removed J3: Conn_01x05, hb44:Pimoroni Haptic Buzz, symbol Connector_Generic:Conn_01x05
- removed J3X1: Conn_01x05, hb44:Pimoroni Haptic Buzz, symbol Connector_Generic:Conn_01x04
- removed J4: Conn_01x02, hb44:TH_BatteryConn, symbol Connector_Generic:Conn_01x02
- removed LCD2: nice!view, hb44:nice!view, symbol hb44:nice!view
- removed LED14, LED15, LED16, LED17, LED18, LED19, LED20, LED21, LED22, LED23, LED24, LED25, LED26, LED27, LED28, LED29, LED30, LED31, LED32, LED33, LED34, LED35, LED36, LED37, LED38, LED39, LED40, LED41, LED42, LED43, LED44, LED45, LED46, LED47, LED48, LED49, LED50: SK6812, hb44:SK6812-SIDE, symbol hb44:SK6812
- removed Q2: Q_PMOS_GSD, hb44:SMD_P_MOSFET_SOT-23, symbol Device:Q_PMOS_GSD
- removed R10, R7, R8, R9: 10k, hb44:SMD_Res_1206, symbol Device:R
- removed R11: 200, hb44:SMD_Res_1206, symbol Device:R
- removed R12: 200k, hb44:SMD_Res_1206, symbol Device:R
- removed SW22, SW23, SW24, SW25, SW26, SW27, SW28, SW29, SW30, SW31, SW32, SW33, SW34, SW35, SW36, SW38, SW39, SW40, SW41, SW42: MX, hb44:SMD_CherryMX_MidHeight_HotSwap, symbol hb44:Switch
- removed SW37: RotaryEncoder_Switch, hb44:EC11, symbol Device:RotaryEncoder_Switch
- removed SW45: SW_DPDT_x2, hb44:SMD_SW_SPDT_PCM12, symbol Switch:SW_DPDT_x2
- removed SW46: SW_PUSH, hb44:SMD_SW_SPST_B3U-3000P-B, symbol kbd:SW_PUSH
- removed U3: nice!nano, hb44:nice!nano, symbol hb44:nice!nano
- removed U4: 74AUP2G14, hb44:SMD_74AUP2G14_SOT-363, symbol hb44:74AUP2G14
- added C10_R1, C11_R1, C12_R1, C13_R1, C14_R1, C15_R1, C1_R1, C2_R1, C3_R1, C4_R1, C5_R1, C6_R1, C7_R1, C8_R1, C9_R1: 0.1u, hb44:SMD_Cap_0603, symbol Device:C
- added D10_R1, D11_R1, D12_R1, D13_R1, D14_R1, D15_R1, D16_R1, D17_R1, D18_R1, D19_R1, D1_R1, D20_R1, D21_R1, D2_R1, D3_R1, D4_R1, D5_R1, D6_R1, D7_R1, D8_R1, D9_R1: (no value), hb44:SMD_SOD123, symbol Device:D_Small
- added H1_R1, H2_R1, H3_R1, H4_R1, H5_R1, H6_R1, H7_R1, H8_R1: MountingHole, hb44:MountingHole_4mm, symbol Mechanical:MountingHole
- added J1_R1: Conn_01x02, hb44:TH_BatteryConn, symbol Connector_Generic:Conn_01x02
- added J2X_R1: Conn_01x05, hb44:Pimoroni Haptic Buzz, symbol Connector_Generic:Conn_01x04
- added J2_R1: Conn_01x05, hb44:Pimoroni Haptic Buzz, symbol Connector_Generic:Conn_01x05
- added LCD1_R1: nice!view, hb44:nice!view, symbol hb44:nice!view
- added LED10_R1, LED11_R1, LED12_R1, LED13_R1, LED5_R1, LED6_R1, LED7_R1, LED8_R1, LED9_R1: SK6812, hb44:WS2812B_data-bridgeable, symbol hb44:SK6812
- added LED1_R1, LED2_R1, LED3_R1, LED4_R1: SK6812, hb44:SK6812-SIDE, symbol hb44:SK6812
- added Q1_R1: Q_PMOS_GSD, hb44:SMD_P_MOSFET_SOT-23, symbol Device:Q_PMOS_GSD
- added R1_R1, R2_R1, R3_R1, R4_R1: 10k, hb44:SMD_Res_1206, symbol Device:R
- added R5_R1: 200, hb44:SMD_Res_1206, symbol Device:R
- added R6_R1: 200k, hb44:SMD_Res_1206, symbol Device:R
- added SW10_R1, SW11_R1, SW12_R1, SW13_R1, SW14_R1, SW15_R1, SW17_R1, SW18_R1, SW19_R1, SW1_R1, SW20_R1, SW21_R1, SW2_R1, SW3_R1, SW4_R1, SW5_R1, SW6_R1, SW7_R1, SW8_R1, SW9_R1: MX, hb44:SMD_CherryMX_MidHeight_HotSwap, symbol hb44:Switch
- added SW16_R1: RotaryEncoder_Switch, hb44:EC11, symbol Device:RotaryEncoder_Switch
- added SW22_R1: SW_DPDT_x2, hb44:SMD_SW_SPDT_PCM12, symbol Switch:SW_DPDT_x2
- added SW23_R1: SW_PUSH, hb44:SMD_SW_SPST_B3U-3000P-B, symbol Switch:SW_Push
- added U1_R1: nice!nano, hb44:nice!nano, symbol hb44:nice!nano
- added U2_R1: 74AUP2G14, hb44:SMD_74AUP2G14_SOT-363, symbol hb44:74AUP2G14
- LED1, LED2, LED3, LED4, LED5, LED6, LED7, LED8, LED9: footprint hb44:SK6812-SIDE -> hb44:WS2812B_data-bridgeable
- SW23: renamed from SW44; symbol kbd:SW_PUSH -> Switch:SW_Push
- renumbered C51 to C14, C52 to C15, J2 to J1, J1 to J2, J1X1 to J2X1, SW43 to SW22
Connections:
- net GND: no longer C13.2, LED13.4 (VSS)
- net GND1: now also C13.2, LED13.4 (VSS)
- net GND3: now also C10_R1.1, C11_R1.2, C12_R1.2, C13_R1.2, C14_R1.2, C15_R1.2, C3_R1.2, C4_R1.2, C5_R1.2, C6_R1.1, C7_R1.1, C8_R1.1, C9_R1.1, J1_R1.2 (Pin_2), J2X_R1.4 (Pin_4), J2_R1.5 (Pin_5), LCD1_R1.4 (GND), LED10_R1.4 (VSS), LED11_R1.4 (VSS), LED12_R1.4 (VSS), LED13_R1.4 (VSS), LED3_R1.4 (VSS), LED4_R1.4 (VSS), LED5_R1.4 (VSS), LED6_R1.4 (VSS), LED7_R1.4 (VSS), LED8_R1.4 (VSS), LED9_R1.4 (VSS), R6_R1.2, SW16_R1.C, SW23_R1.2, U1_R1.23 (GND3), U2_R1.2 (GND3)
- net col0: now also U1.15 (P1.11/L); no longer U1.16 (P1.13/L)
- net col1: now also U1.14 (P0.10/L); no longer U1.15 (P1.11/L)
- net col2: now also U1.13 (P0.09/L); no longer U1.14 (P0.10/L)
- net col3: now also U1.11 (P1.04/L); no longer U1.13 (P0.09/L)
- net rotA: now also U1.16 (P1.13/L); no longer U1.12 (P1.06/L)
- net rotB: now also U1.17 (P1.15/L); no longer U1.11 (P1.04/L)
- net row1: now also U1.18 (P0.02/L); no longer U1.19 (P0.29/L)
- net row2: now also U1.12 (P1.06/L); no longer U1.18 (P0.02/L)
- net row3: now also U1.19 (P0.29/L); no longer U1.17 (P1.15/L)
- net +3V3 renamed VCC
- new net: D21_R1.2 (A), SW21_R1.2 (ROW)
- new net: D10_R1.2 (A), SW10_R1.2 (ROW)
- new net: R1_R1.2, R3_R1.1, SW16_R1.A
- new net: R2_R1.2, R4_R1.1, SW16_R1.B
- new net: LED4_R1.3 (DOUT), LED5_R1.1 (DIN)
- new net: LED5_R1.3 (DOUT), LED6_R1.1 (DIN)
- new net: D11_R1.2 (A), SW11_R1.2 (ROW)
- new net: C14_R1.1, R3_R1.2, U2_R1.1
- new net: D3_R1.2 (A), SW3_R1.2 (ROW)
- new net: LED6_R1.3 (DOUT), LED7_R1.1 (DIN)
- new net: D20_R1.2 (A), SW20_R1.2 (ROW)
- new net: D9_R1.2 (A), SW9_R1.2 (ROW)
- new net: D6_R1.2 (A), SW6_R1.2 (ROW)
- new net: C15_R1.1, R4_R1.2, U2_R1.3
- new net: LED7_R1.3 (DOUT), LED8_R1.1 (DIN)
- new net: D14_R1.2 (A), SW14_R1.2 (ROW)
- new net: D5_R1.2 (A), SW5_R1.2 (ROW)
- new net: LED2_R1.3 (DOUT), LED3_R1.1 (DIN)
- new net: LED3_R1.3 (DOUT), LED4_R1.1 (DIN)
- new net: D4_R1.2 (A), SW4_R1.2 (ROW)
- new net: D12_R1.2 (A), SW12_R1.2 (ROW)
- new net: D1_R1.2 (A), SW1_R1.2 (ROW)
- new net: D2_R1.2 (A), SW2_R1.2 (ROW)
- new net: D18_R1.2 (A), SW18_R1.2 (ROW)
- new net: LED8_R1.3 (DOUT), LED9_R1.1 (DIN)
- new net: LED1_R1.3 (DOUT), LED2_R1.1 (DIN)
- new net: D7_R1.2 (A), SW7_R1.2 (ROW)
- new net: Q1_R1.1 (G), R5_R1.2
- new net: D8_R1.2 (A), SW8_R1.2 (ROW)
- new net: D15_R1.2 (A), SW15_R1.2 (ROW)
- new net: D19_R1.2 (A), SW19_R1.2 (ROW)
- new net: D17_R1.2 (A), SW17_R1.2 (ROW)
- new net: LED10_R1.1 (DIN), LED9_R1.3 (DOUT)
- new net: LED11_R1.3 (DOUT), LED12_R1.1 (DIN)
- new net: LED12_R1.3 (DOUT), LED13_R1.1 (DIN)
- new net: D13_R1.2 (A), SW13_R1.2 (ROW)
- new net: LED10_R1.3 (DOUT), LED11_R1.1 (DIN)
- new net ARGB_R: LED1_R1.1 (DIN), U1_R1.1 (P0.06/H)
- new net CS_R: LCD1_R1.5 (CS), U1_R1.5 (P0.17/H)
- new net GND2: C1_R1.2, C2_R1.2, LED1_R1.4 (VSS), LED2_R1.4 (VSS), U1_R1.3 (GND2), U1_R1.4 (GND2)
- new net LED_R: R5_R1.1, R6_R1.1, U1_R1.2 (P0.08/H)
- new net LED_VCC_R: C10_R1.2, C11_R1.1, C12_R1.1, C13_R1.1, C1_R1.1, C2_R1.1, C3_R1.1, C4_R1.1, C5_R1.1, C6_R1.2, C7_R1.2, C8_R1.2, C9_R1.2, LED10_R1.2 (VDD), LED11_R1.2 (VDD), LED12_R1.2 (VDD), LED13_R1.2 (VDD), LED1_R1.2 (VDD), LED2_R1.2 (VDD), LED3_R1.2 (VDD), LED4_R1.2 (VDD), LED5_R1.2 (VDD), LED6_R1.2 (VDD), LED7_R1.2 (VDD), LED8_R1.2 (VDD), LED9_R1.2 (VDD), Q1_R1.3 (D)
- new net MOSI_R: LCD1_R1.1 (MOSI), U1_R1.7 (P0.22/H)
- new net RAW_BAT_R: J1_R1.1 (Pin_1), SW22_R1.1 (A)
- new net RAW_R: SW22_R1.2 (B), U1_R1.24 (BAT+)
- new net RESET_R: SW23_R1.1, U1_R1.22 (RESET)
- new net SCK_R: LCD1_R1.2 (SCK), U1_R1.6 (P0.20/H)
- new net SCL/RX_R: J2X_R1.3 (Pin_3), J2_R1.3 (Pin_3), U1_R1.8 (P0.24/H)
- new net SDA/TX_R: J2X_R1.2 (Pin_2), J2_R1.2 (Pin_2), J2_R1.4 (Pin_4), U1_R1.9 (P1.00/H)
- new net VDD: J2X_R1.1 (Pin_1), J2_R1.1 (Pin_1), LCD1_R1.3 (VCC), Q1_R1.2 (S), R1_R1.1, R2_R1.1, U1_R1.21 (3.3V), U2_R1.5 (VDD)
- new net col0_R: SW11_R1.1 (COL), SW1_R1.1 (COL), SW21_R1.1 (COL), SW6_R1.1 (COL), U1_R1.10 (P0.11/H)
- new net col1_R: SW12_R1.1 (COL), SW16_R1.S1, SW2_R1.1 (COL), SW7_R1.1 (COL), U1_R1.13 (P0.09/L)
- new net col2_R: SW13_R1.1 (COL), SW17_R1.1 (COL), SW3_R1.1 (COL), SW8_R1.1 (COL), U1_R1.20 (P0.31/L)
- new net col3_R: SW14_R1.1 (COL), SW18_R1.1 (COL), SW4_R1.1 (COL), SW9_R1.1 (COL), U1_R1.19 (P0.29/L)
- new net col4_R: SW10_R1.1 (COL), SW15_R1.1 (COL), SW19_R1.1 (COL), SW5_R1.1 (COL), U1_R1.18 (P0.02/L)
- new net col5_R: SW20_R1.1 (COL), U1_R1.27 (P1.07/L)
- new net rotA_R: U1_R1.12 (P1.06/L), U2_R1.6
- new net rotB_R: U1_R1.11 (P1.04/L), U2_R1.4
- new net rotS2_R: D16_R1.2 (A), SW16_R1.S2
- new net row0_R: D1_R1.1 (K), D2_R1.1 (K), D3_R1.1 (K), D4_R1.1 (K), D5_R1.1 (K), U1_R1.16 (P1.13/L)
- new net row1_R: D10_R1.1 (K), D6_R1.1 (K), D7_R1.1 (K), D8_R1.1 (K), D9_R1.1 (K), U1_R1.17 (P1.15/L)
- new net row2_R: D11_R1.1 (K), D12_R1.1 (K), D13_R1.1 (K), D14_R1.1 (K), D15_R1.1 (K), U1_R1.15 (P1.11/L)
- new net row3_R: D16_R1.1 (K), D17_R1.1 (K), D18_R1.1 (K), D19_R1.1 (K), D20_R1.1 (K), D21_R1.1 (K), U1_R1.14 (P0.10/L)
Other:
- note added: "-9+4 Individually addressible RGB LEDs -Decoupled with 0.1uF capacitors -Toggled with mosfet for power savings"
- note added: "-waveshare 20903 via UART -mutually exclusive with haptic"
- note removed: "-22 Individually addressible RGB LEDs -Decoupled with 0.1uF capacitors -Toggled with mosfet for power savings"
- note removed: "-adafruit 4750 and uses UART -mutually exclusive with haptic"
- moved on the sheet: C14, C15, H1, H2, H3, H4, H5, H6, H7, H8, J2, J2X1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
